File: newrev.brd (EAGLE design)
At the start: 204.4 x 88.6 mm, 134 parts, among them IC1 P82B715D, J1 6473427-1, J2 VR10S05, Q1 MOSFET-NCHANNELSMD, Q2 MOSFET-NCHANNELSMD, SW1 CTS_ELECTROCOMPONENTS_204-211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, SW2 CTS_ELECTROCOMPONENTS_204-211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, U1 XC6220B331MR-G, U4 ARDUINO_R3_SHIELD, U6 ADS1119IPWT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

Commit message: Revised LEDs
Changed LED pins on Arduino Mega (will need to adjust program accordingly)
Reorganized LED pins
Placed LEDs and corresponding resistors on board
Parts:
- moved R71 780.4 mm to (105.4, 62.2), flipped to the bottom, turned to 180 degrees
- moved C1 684.6 mm to (-47.0, 15.2)
- moved C11 684.6 mm to (-47.0, -25.4)
- moved C13 684.6 mm to (-47.0, -33.0)
- moved C15 684.6 mm to (-47.0, -40.6)
- moved C17 684.6 mm to (-47.0, -48.3)
- moved C19 684.6 mm to (-47.0, -55.9)
- moved C21 684.6 mm to (-47.0, -63.5)
- moved C23 684.6 mm to (-47.0, -71.1)
- moved C26 684.6 mm to (-47.0, -82.5)
- moved C28 684.6 mm to (-47.0, -90.2)
- moved C3 684.6 mm to (-47.0, 6.35)
- moved C30 684.6 mm to (-47.0, -97.8)
- moved C32 684.6 mm to (-47.0, -105.4)
- moved C34 684.6 mm to (-47.0, -113.0)
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Connections:
- net 10: now also LAMBDAS.4; no longer BRAKETEMP.2
- net 15: now also BRAKETEMP.2; no longer BRAKETEMP.4
- net 16: now also SHOCKPOT.4; no longer SHOCKPOT.2
- net 18: now also SHOCKPOT.2; no longer SHOCKPOT.4
- net 19: now also BRAKEPRES.4; no longer BRAKEPRES.2
- net 23: now also BRAKEPRES.2; no longer BRAKEPRES.4
- net 24: now also INTAKEPRES.4; no longer INTAKEPRES.2
- net 26: now also INTAKEPRES.2; no longer INTAKEPRES.4
- net 27: now also INTAKETEMP.4; no longer INTAKETEMP.2
- net 29: now also INTAKETEMP.2; no longer INTAKETEMP.4
- net 30: now also COOLANTTEMP.4; no longer COOLANTTEMP.2
- net 32: now also COOLANTTEMP.2; no longer COOLANTTEMP.4
- net 33: now also OILPRES.4; no longer OILPRES.2
- net 35: now also OILPRES.2; no longer OILPRES.4
- net 36: now also OILTEMP.4; no longer OILTEMP.2
- net 38: now also OILTEMP.2; no longer OILTEMP.4
- net 39: now also SPARE1.4; no longer SPARE1.2
- net 4: now also BRAKETEMP.4; no longer DASH.2
- net 41: now also SPARE1.2; no longer SPARE1.4
- net 42: now also SPARE2.4; no longer SPARE2.2
- net 44: now also SPARE2.2; no longer SPARE2.4
- net 45: now also DAQ.4; no longer DAQ.2
- net 47: now also DAQ.2; no longer DAQ.4
- net 5: now also DASH.2; no longer DASH.3
- net 6: now also DASH.3; no longer DASH.4
- net 7: now also DASH.4; no longer LAMBDAS.2
- net 8: now also LAMBDAS.2; no longer LAMBDAS.3
- net 9: now also LAMBDAS.3; no longer LAMBDAS.4
Routing:
- net 5V: track 51.6 -> 184.8 mm, vias 5 -> 4
- net 48: track 147.9 -> 74.0 mm, vias 3 -> 1
- net REC: track 89.5 -> 162.6 mm, vias 2 -> 0
- net 34: track 31.0 -> 90.8 mm, vias 2 -> 0
- net 33: track 26.6 -> 85.9 mm, vias 2 -> 0
- net 26: track 20.8 -> 77.1 mm
- net 24: track 19.2 -> 74.6 mm
- net 9: track 89.7 -> 143.6 mm, vias 1 -> 0
- net 25: track 19.9 -> 72.9 mm
- net 8: track 87.7 -> 140.7 mm, vias 1 -> 0
- net 35: track 37.0 -> 88.4 mm, vias 4 -> 0
- net 6: track 73.9 -> 123.2 mm, vias 1 -> 0
- net 5: track 71.7 -> 120.4 mm, vias 1 -> 0
- net 7: track 78.8 -> 125.1 mm, vias 1 -> 0
- net 23: track 36.4 -> 81.8 mm, vias 2 -> 0
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