File: newrev.sch (EAGLE design)
At the start: 134 parts, among them IC1 P82B715D, J1 6473427-1, J2 VR10S05, Q1 MOSFET-NCHANNELSMD, Q2 MOSFET-NCHANNELSMD, SW1 CTS_ELECTROCOMPONENTS_204-211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, SW2 CTS_ELECTROCOMPONENTS_204-211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, U1 XC6220B331MR-G, U4 ARDUINO_R3_SHIELD, U6 ADS1119IPWT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

Commit message: Revised LEDs
Changed LED pins on Arduino Mega (will need to adjust program accordingly)
Reorganized LED pins
Placed LEDs and corresponding resistors on board
Connections:
- net 10: now also LAMBDAS.K_GREEN; no longer BRAKETEMP.K_BLUE
- net 15: now also BRAKETEMP.K_BLUE; no longer BRAKETEMP.K_GREEN
- net 16: now also SHOCKPOT.K_GREEN; no longer SHOCKPOT.K_BLUE
- net 18: now also SHOCKPOT.K_BLUE; no longer SHOCKPOT.K_GREEN
- net 19: now also BRAKEPRES.K_GREEN; no longer BRAKEPRES.K_BLUE
- net 23: now also BRAKEPRES.K_BLUE; no longer BRAKEPRES.K_GREEN
- net 24: now also INTAKEPRES.K_GREEN; no longer INTAKEPRES.K_BLUE
- net 26: now also INTAKEPRES.K_BLUE; no longer INTAKEPRES.K_GREEN
- net 27: now also INTAKETEMP.K_GREEN; no longer INTAKETEMP.K_BLUE
- net 29: now also INTAKETEMP.K_BLUE; no longer INTAKETEMP.K_GREEN
- net 30: now also COOLANTTEMP.K_GREEN; no longer COOLANTTEMP.K_BLUE
- net 32: now also COOLANTTEMP.K_BLUE; no longer COOLANTTEMP.K_GREEN
- net 33: now also OILPRES.K_GREEN; no longer OILPRES.K_BLUE
- net 35: now also OILPRES.K_BLUE; no longer OILPRES.K_GREEN
- net 36: now also OILTEMP.K_GREEN; no longer OILTEMP.K_BLUE
- net 38: now also OILTEMP.K_BLUE; no longer OILTEMP.K_GREEN
- net 39: now also SPARE1.K_GREEN; no longer SPARE1.K_BLUE
- net 4: now also BRAKETEMP.K_GREEN; no longer DASH.K_BLUE
- net 41: now also SPARE1.K_BLUE; no longer SPARE1.K_GREEN
- net 42: now also SPARE2.K_GREEN; no longer SPARE2.K_BLUE
- net 44: now also SPARE2.K_BLUE; no longer SPARE2.K_GREEN
- net 45: now also DAQ.K_GREEN; no longer DAQ.K_BLUE
- net 47: now also DAQ.K_BLUE; no longer DAQ.K_GREEN
- net 5: now also DASH.K_BLUE; no longer DASH.K_RED
- net 6: now also DASH.K_RED; no longer DASH.K_GREEN
- net 7: now also DASH.K_GREEN; no longer LAMBDAS.K_BLUE
- net 8: now also LAMBDAS.K_BLUE; no longer LAMBDAS.K_RED
- net 9: now also LAMBDAS.K_RED; no longer LAMBDAS.K_GREEN
